File: schematic/SZBK07.sch (KiCad schematic (older format))
At the start: 22 parts, among them Q1 2N7000, Q2 2N7000, Q3 PSMN3R3-80PS, U1 SZBK07_DC-DC_module, U2 AD822A, U3 MP2307_DC-DC_module, U4 ArduinoNano

Commit message: R1 added, error in original
Parts:
- removed U3: MP2307_DC-DC_module, symbol MP2307_DC-DC_module
- added R1: 100K, symbol Device:R
- added U3: MP2307_DC-DC_module, symbol Modules:MP2307_DC-DC_module
- BT1: symbol Battery -> Device:Battery
- C1: value C -> 0.1uF; symbol C -> Device:C
- C2: symbol C -> Device:C
- D1: symbol D_Zener_ALT -> Device:D_Zener_ALT
- D4: symbol D_ALT -> Device:D_ALT
- Q1, Q2: symbol 2N7000 -> Modules:2N7000
- Q3: symbol IRFZ44N -> Modules:IRFZ44N
- R10, R2, R3, R4, R5, R6, R7, R8, R9: symbol R -> Device:R
- SC1: symbol Solar_Cells -> Device:Solar_Cells
- U1: symbol SZBK07_DC-DC_module -> Modules:SZBK07_DC-DC_module
- U2: symbol AD822A -> Modules:AD822A
- U4: symbol ArduinoNano -> Modules:ArduinoNano
Connections:
- net +7V: now also U3.4 (OUT+)
- net ArduinoPin_A2: no longer C2.1
- net GND: now also U3.2 (IN-), U3.3 (OUT-)
- net Vbb: now also U3.1 (IN+)
- net Vpp: now also R1.2; no longer D1.1 (K), R3.1
- net at R2.1: now also R3.1, R1.1
Changed lines of the file:
@@
-EESchema Schematic File Version 2
-LIBS:Modules
-LIBS:power
-LIBS:device
-LIBS:switches
-LIBS:relays
-LIBS:motors
-LIBS:transistors
-LIBS:conn
-LIBS:linear
-LIBS:regul
-LIBS:74xx
-LIBS:cmos4000
-LIBS:adc-dac
-LIBS:memory
-LIBS:xilinx
-LIBS:microcontrollers
-LIBS:dsp
-LIBS:microchip
-LIBS:analog_switches
-LIBS:motorola
-LIBS:texas
-LIBS:intel
-LIBS:audio
-LIBS:interface
-LIBS:digital-audio
-LIBS:philips
-LIBS:display
-LIBS:cypress
-LIBS:siliconi
-LIBS:opto
-LIBS:atmel
-LIBS:contrib
-LIBS:valves
+EESchema Schematic File Version 4
 LIBS:SZBK07-cache
-EELAYER 25 0
+EELAYER 26 0
 EELAYER END
 $Descr A4 11693 8268
@@
 $EndDescr
 $Comp
-L SZBK07_DC-DC_module U1
+L Modules:SZBK07_DC-DC_module U1
 U 1 1 5B485D2D
 P 3950 3250
@@
 $EndComp
 $Comp
-L GNDPWR #PWR2
+L power:GNDPWR #PWR02
 U 1 1 5B485E0B
 P 2400 2650
-F 0 "#PWR2" H 2400 2450 50  0001 C CNN
+F 0 "#PWR02" H 2400 2450 50  0001 C CNN
 F 1 "GNDPWR" H 2400 2500 50  0000 C CNN
 F 2 "" H 2400 2600 50  0001 C CNN
@@
 $EndComp
 $Comp
-L Solar_Cells SC1
+L Device:Solar_Cells SC1
 U 1 1 5B485E23
 P 1250 3200
@@
 Vpp
 $Comp
-L IRFZ44N Q3
+L Modules:IRFZ44N Q3
 U 1 1 5B485EB4
 P 6550 2700
@@
 	5975 2800 6350 2800
 $Comp
-L Battery BT1
+L Device:Battery BT1
 U 1 1 5B485F93
 P 8850 3100
@@
 $EndComp
 $Comp
-L GNDPWR #PWR3
+L power:GNDPWR #PWR03
 U 1 1 5B485FBA
 P 8850 3300
-F 0 "#PWR3" H 8850 3100 50  0001 C CNN
+F 0 "#PWR03" H 8850 3100 50  0001 C CNN
 F 1 "GNDPWR" H 8850 3170 50  0000 C CNN
 F 2 "" H 8850 3250 50  0001 C CNN
@@
 	6650 1750 6650 2300
 $Comp
-L R R2
+L Device:R R2
 U 1 1 5B4865B4
 P 5975 1500
@@
 	5975 1750 5975 2025
 $Comp
-L R R3
+L Device:R R3
 U 1 1 5B48662F
 P 6950 1500
@@
 Wire Wire Line
 	6950 1750 6950 2025
-Wire Wire Line
-	5800 1350 6950 1350
-Wire Wire Line
-	6950 1350 7450 1350
-$Comp
-L D_Zener_ALT D1
+$Comp
+L Device:D_Zener_ALT D1
 U 1 1 5B4866B2
 P 7450 2400
@@
 Wire Wire Line
 	7450 1350 7450 2250
-Connection ~ 6950 1350
-Wire Wire Line
-	5800 1350 1750 1350
 Wire Wire Line
 	1750 1350 1750 2900
 $Comp
-L AD822A U2
+L Modules:AD822A U2
 U 1 1 5B48809D
 P 3800 4200
@@
 $EndComp
 $Comp
-L GND #PWR1
+L power:GND #PWR01
 U 1 1 5B488158
 P 2050 2650
-F 0 "#PWR1" H 2050 2400 50  0001 C CNN
+F 0 "#PWR01" H 2050 2400 50  0001 C CNN
 F 1 "GND" H 2050 2500 50  0000 C CNN
 F 2 "" H 2050 2650 50  0001 C CNN
@@
 $EndComp
 $Comp
-L GND #PWR5
+L power:GND #PWR05
 U 1 1 5B4881AE
 P 3700 4650
-F 0 "#PWR5" H 3700 4400 50  0001 C CNN
+F 0 "#PWR05" H 3700 4400 50  0001 C CNN
 F 1 "GND" H 3700 4500 50  0000 C CNN
 F 2 "" H 3700 4650 50  0001 C CNN
@@
 	3350 4100 3500 4100
 $Comp
-L R R7
+L Device:R R7
 U 1 1 5B48878B
 P 3200 4150
@@
 	3700 4500 3700 4650
 $Comp
-L R R8
+L Device:R R8
 U 1 1 5B48887F
 P 4400 4450
@@
 Wire Wire Line
 	4400 4950 3200 4950
-Connection ~ 3200 4300
 Text GLabel 4400 4200 2    60   Input ~ 0
 ArduinoPin_A1
 $Comp
-L R R5
+L Device:R R5
 U 1 1 5B488988
 P 2200 4100
@@
 $EndComp
 $Comp
-L R R9
+L Device:R R9
 U 1 1 5B4889C5
 P 2500 4650
@@
 $EndComp
 $Comp
-L GND #PWR6
+L power:GND #PWR06
 U 1 1 5B488A20
 P 2500 4900
-F 0 "#PWR6" H 2500 4650 50  0001 C CNN
+F 0 "#PWR06" H 2500 4650 50  0001 C CNN
 F 1 "GND" H 2500 4750 50  0000 C CNN
 F 2 "" H 2500 4900 50  0001 C CNN
@@
 ArduinoPin_A0
 $Comp
-L C C1
+L Device:C C1
 U 1 1 5B488DB5
 P 2200 4550
 F 0 "C1" H 2225 4650 50  0000 L CNN
-F 1 "C" H 2225 4450 50  0000 L CNN
+F 1 "0.1uF" H 2225 4450 50  0000 L CNN
 F 2 "" H 2238 4400 50  0001 C CNN
 F 3 "" H 2200 4550 50  0001 C CNN
@@
 Connection ~ 2200 4400
 $Comp
-L R R6
+L Device:R R6
 U 1 1 5B489033
 P 5950 4200
@@
 $EndComp
 $Comp
-L R R10
+L Device:R R10
 U 1 1 5B489039
 P 5950 4650
@@
 $EndComp
 $Comp
-L GND #PWR7
+L power:GND #PWR07
 U 1 1 5B48903F
 P 5950 4900
-F 0 "#PWR7" H 5950 4650 50  0001 C CNN
+F 0 "#PWR07" H 5950 4650 50  0001 C CNN
 F 1 "GND" H 5950 4750 50  0000 C CNN
 F 2 "" H 5950 4900 50  0001 C CNN
@@
 ArduinoPin_A2
 $Comp
-L C C2
+L Device:C C2
 U 1 1 5B489048
 P 5650 4550
@@
 	1    0    0    -1
 $EndComp
-Wire Wire Line
-	5350 4400 5650 4400
-Wire Wire Line
-	5650 4400 5950 4400
 Connection ~ 5950 4400
 Wire Wire Line
@@
 Wire Wire Line
 	5650 4900 5950 4900
-Connection ~ 5650 4400
-$Comp
-L D_ALT D4
+$Comp
+L Device:D_ALT D4
 U 1 1 5B48ABB8
 P 5000 3750
@@
 $EndComp
 $Comp
-L R R4
+L Device:R R4
 U 1 1 5B48ACD1
 P 4750 3900
@@
 Wire Wire Line
 	7450 2800 7450 2550
-$Comp
-L MP2307_DC-DC_module U3
-U 1 1 5B48BDD1
-P 2500 6000
-F 0 "U3" H 2400 6110 60  0000 C CNN
-F 1 "MP2307_DC-DC_module" H 2390 6260 60  0000 C CNN
-F 2 "" H 2500 5950 60  0001 C CNN
-F 3 "" H 2500 5950 60  0001 C CNN
-	1    2500 6000
-	1    0    0    -1
-$EndComp
-Text GLabel 1500 5600 0    60   Input ~ 0
+Text GLabel 1850 5600 0    60   Input ~ 0
 Vbb
-Text GLabel 3300 5600 2    60   Input ~ 0
+Text GLabel 2850 5600 2    60   Input ~ 0
 +7V
 $Comp
-L GND #PWR10
+L power:GND #PWR010
 U 1 1 5B48C726
-P 1500 5900
-F 0 "#PWR10" H 1500 5650 50  0001 C CNN
-F 1 "GND" H 1500 5750 50  0000 C CNN
-F 2 "" H 1500 5900 50  0001 C CNN
-F 3 "" H 1500 5900 50  0001 C CNN
-	1    1500 5900
-	1    0    0    -1
-$EndComp
-$Comp
-L GND #PWR11
+P 1850 5900
+F 0 "#PWR010" H 1850 5650 50  0001 C CNN
+F 1 "GND" H 1850 5750 50  0000 C CNN
+F 2 "" H 1850 5900 50  0001 C CNN
+F 3 "" H 1850 5900 50  0001 C CNN
+	1    1850 5900
+	1    0    0    -1
+$EndComp
+$Comp
+L power:GND #PWR011
 U 1 1 5B48C76A
-P 3300 5900
-F 0 "#PWR11" H 3300 5650 50  0001 C CNN
-F 1 "GND" H 3300 5750 50  0000 C CNN
-F 2 "" H 3300 5900 50  0001 C CNN
-F 3 "" H 3300 5900 50  0001 C CNN
-	1    3300 5900
-	1    0    0    -1
-$EndComp
-$Comp
-L ArduinoNano U4
+P 2850 5900
+F 0 "#PWR011" H 2850 5650 50  0001 C CNN
+F 1 "GND" H 2850 5750 50  0000 C CNN
+F 2 "" H 2850 5900 50  0001 C CNN
+F 3 "" H 2850 5900 50  0001 C CNN
+	1    2850 5900
+	1    0    0    -1
+$EndComp
+$Comp
+L Modules:ArduinoNano U4
 U 1 1 5B48C7AE
 P 4400 6150
@@
 +5V
 $Comp
-L GND #PWR9
+L power:GND #PWR09
 U 1 1 5B48CCA3
 P 3700 5750
-F 0 "#PWR9" H 3700 5500 50  0001 C CNN
+F 0 "#PWR09" H 3700 5500 50  0001 C CNN
 F 1 "GND" H 3700 5600 50  0000 C CNN
 F 2 "" H 3700 5750 50  0001 C CNN
@@
 $EndComp
 $Comp
-L GND #PWR8
+L power:GND #PWR08
 U 1 1 5B48CCF9
 P 5150 5550
-F 0 "#PWR8" H 5150 5300 50  0001 C CNN
+F 0 "#PWR08" H 5150 5300 50  0001 C CNN
 F 1 "GND" H 5150 5400 50  0000 C CNN
 F 2 "" H 5150 5550 50  0001 C CNN
@@
 	2650 2800 2650 2650
 $Comp
-L GND #PWR4
+L power:GND #PWR04
 U 1 1 5B494DA1
 P 3350 4100
-F 0 "#PWR4" H 3350 3850 50  0001 C CNN
+F 0 "#PWR04" H 3350 3850 50  0001 C CNN
 F 1 "GND" H 3350 3950 50  0000 C CNN
 F 2 "" H 3350 4100 50  0001 C CNN
@@
 12V BATTERY\nFLA, AGM OR Lithium
 $Comp
-L 2N7000 Q2
+L Modules:2N7000 Q2
 U 1 1 5B5C69A6
 P 6850 2225
@@
 $EndComp
 $Comp
-L 2N7000 Q1
+L Modules:2N7000 Q1
 U 1 1 5B5C6A55
 P 6075 2225
@@
 	6650 2300 6275 2300
 Connection ~ 5975 1750
+Wire Wire Line
+	5350 4400 5950 4400
+$Comp
+L Modules:MP2307_DC-DC_module U3
+U 1 1 5C31A193
+P 2350 6000
+F 0 "U3" H 2350 6745 60  0000 C CNN
+F 1 "MP2307_DC-DC_module" H 2350 6635 60  0000 C CNN
+F 2 "" H 2350 5950 60  0001 C CNN
+F 3 "" H 2350 5950 60  0001 C CNN
+	1    2350 6000
+	1    0    0    -1
+$EndComp
+$Comp
+L Device:R R1
+U 1 1 5C31D36F
+P 5600 1350
+F 0 "R1" V 5500 1350 50  0000 C CNN
+F 1 "100K" V 5600 1350 50  0000 C CNN
+F 2 "" V 5530 1350 50  0001 C CNN
+F 3 "~" H 5600 1350 50  0001 C CNN
+	1    5600 1350
+	0    1    1    0
+$EndComp
+Wire Wire Line
+	5750 1350 5975 1350
+Connection ~ 5975 1350
+Wire Wire Line
+	5975 1350 6950 1350
+Wire Wire Line
+	5450 1350 1750 1350
 $EndSCHEMATC

Commit message: R1 added, error fixed
Connections:
- net at R1.1, R2.1, R3.1: now also D1.1 (K)
Changed lines of the file:
@@
 Wire Wire Line
 	5450 1350 1750 1350
+Wire Wire Line
+	6950 1350 7450 1350
+Connection ~ 6950 1350
 $EndSCHEMATC
