File: schematic_18/SZBK07_18.sch (KiCad schematic (older format))
At the start: 23 parts, among them Q1 2N7000, Q2 2N7000, Q3 PSMN3R3-80PS, U1 SZBK07_DC-DC_module, U2 AD822A, U3 MP2307_DC-DC_module, U4 ArduinoNano

Commit message: revised with 2 versions for 18V and 30V panels
Parts:
- removed D1: 1N4742, symbol Device:D_Zener_ALT
- removed Q1, Q2: 2N7000, TO_SOT_Packages_THT:TO-92_Molded_Narrow, symbol Modules:2N7000
- removed Q3: PSMN3R3-80PS, TO-220, symbol Modules:IRFZ44N
- removed R1: 100K, symbol Device:R
- added D? (x2): D_ALT, symbol Device:D_ALT
- added Q?: IRF4905, TO-220, symbol Modules:IRF4905
- added Q? (x2): 2N3906, Package_TO_SOT_THT:TO-92_Inline, symbol Transistor_BJT:2N3906
Connections:
- wire segments 71 -> 56
Other:
- note added: "SOLAR PANEL\n0 TO 25v"
- note added: "This circuit is intended for use with a 36-cell solar panel (MPP voltage of 18V)."
- note removed: "SOLAR PANEL\n0 TO 40v"
- moved on the sheet: BT1, R2, R3
